File: ButtonBoards/6ButtonSMD/6ButtonSMD.brd (EAGLE design)
At the start: 48.3 x 66 mm, 20 parts, among them J1 4P-SMD-2.0-90D

Commit message: smd
Parts:
- moved J1 2.16 mm to (27.6, -56.8)
Routing:
- net GND: track 0.00 -> 78.3 mm
- net N$30: track 0.00 -> 43.0 mm
- net N$27: track 0.00 -> 36.4 mm
- net A: track 0.00 -> 27.2 mm
- net +5V: track 0.00 -> 12.0 mm
- net +3V3: track 0.00 -> 7.85 mm
- net N$6: track 0.00 -> 6.86 mm
- net N$4: track 0.00 -> 6.86 mm
- net N$2: track 0.00 -> 5.59 mm
- net N$3: track 0.00 -> 5.51 mm
- net N$1: track 0.00 -> 5.51 mm
- net N$5: track 0.00 -> 4.24 mm
